Commit message: Fixed moveit pack and added the gripper

File: robot_model/urdf/gripper.xacro (robot description, xacro)
@@ -1,21 +1,14 @@
 <?xml version="1.0" ?>
-<!-- =================================================================================== -->
-<!-- |    This document was autogenerated by xacro from Downloads/Gripper_Closed_1v2/urdf/Gripper_Closed_1v2.urdf | -->
-<!-- |    EDITING THIS FILE BY HAND IS NOT RECOMMENDED                                 | -->
-<!-- =================================================================================== -->
-<!-- This URDF was automatically created by SolidWorks to URDF Exporter! Originally created by Stephen Brawner (brawner@gmail.com)
-     Commit Version: 1.5.1-0-g916b5db  Build Version: 1.5.7152.31018
-     For more information, please see http://wiki.ros.org/sw_urdf_exporter -->
-<robot name="Gripper_Closed_1v2">
-  <link name="gripper_body">robot_description
+<robot xmlns:xacro="http://www.ros.org/wiki/xacro" name="ur5">
+  <link name="gripper_body">
     <inertial>
-      <origin rpy="0 0 0" xyz="2.9342E-05 -0.044291 0.00032345"/>
+      <origin xyz="2.9342E-05 -0.044291 0.00032345" rpy="0 0 0"/>
       <mass value="0.47636"/>
       <inertia ixx="0.00034357" ixy="-3.8819E-08" ixz="3.6487E-08" iyy="0.00014964" iyz="7.9271E-06" izz="0.00038471"/>
     </inertial>
     <visual>
-      <origin rpy="0 0 0" xyz="0 0 0"/>
+      <origin xyz="0 0 0" rpy="0 0 0"/>
       <geometry>
-        <mesh filename="package://robot_model/meshes/gripper/ee_link.STL"/>
+        <mesh filename="package://robot_model/meshes/gripper/gripper_body.STL"/>
       </geometry>
       <material name="">
@@ -24,7 +17,7 @@
     </visual>
     <collision>
-      <origin rpy="0 0 0" xyz="0 0 0"/>
+      <origin xyz="0 0 0" rpy="0 0 0"/>
       <geometry>
-        <mesh filename="package://robot_model/meshes/gripper/ee_link.STL"/>
+        <mesh filename="package://robot_model/meshes/gripper/gripper_body.STL"/>
       </geometry>
     </collision>

File: robot_model/urdf/lego_bot.xacro (robot description, xacro)
@@ -33,5 +33,5 @@
     <parent link="gripper_body" />
     <child link = "TCP" />
-    <origin xyz="0.0 -0.233 -0.01905" rpy="3.14159265359 1.57079632679 -1.57079632679" />
+    <origin xyz="0.0 -0.264 0.0" rpy="3.14159265359 1.57079632679 -1.57079632679" />
   </joint>
   <!-- Realsense Cam -->

Commit message: Added the new URDF file and meshes. Used the newest uploaded gripper, but didnt doublecheck the distance fit. Head hurt, and couldnt overskue det

File: robot_model/urdf/gripper.xacro (robot description, xacro)
@@ -3,10 +3,10 @@
   <link name="gripper_body">
     <inertial>
-      <origin xyz="2.9342E-05 -0.044291 0.00032345" rpy="0 0 0"/>
-      <mass value="0.47636"/>
-      <inertia ixx="0.00034357" ixy="-3.8819E-08" ixz="3.6487E-08" iyy="0.00014964" iyz="7.9271E-06" izz="0.00038471"/>
+      <origin rpy="0 0 0" xyz="2.1478E-05 -0.056983 0.0015312"/>
+      <mass value="0.44225"/>
+      <inertia ixx="0.00031483" ixy="-3.882E-08" ixz="3.7547E-08" iyy="0.00016784" iyz="6.6712E-06" izz="0.00035617"/>
     </inertial>
     <visual>
-      <origin xyz="0 0 0" rpy="0 0 0"/>
+      <origin rpy="0 0 0" xyz="0 0 0"/>
       <geometry>
         <mesh filename="package://robot_model/meshes/gripper/gripper_body.STL"/>
@@ -17,5 +17,5 @@
     </visual>
     <collision>
-      <origin xyz="0 0 0" rpy="0 0 0"/>
+      <origin rpy="0 0 0" xyz="0 0 0"/>
       <geometry>
         <mesh filename="package://robot_model/meshes/gripper/gripper_body.STL"/>

Commit message: New gripper added

File: robot_model/urdf/gripper.xacro (robot description, xacro)
@@ -3,23 +3,23 @@
   <link name="gripper_body">
     <inertial>
-      <origin xyz="2.9342E-05 -0.044291 0.00032345" rpy="0 0 0"/>
-      <mass value="0.47636"/>
-      <inertia ixx="0.00034357" ixy="-3.8819E-08" ixz="3.6487E-08" iyy="0.00014964" iyz="7.9271E-06" izz="0.00038471"/>
+      <origin xyz="2.1478E-05 -0.056983 0.0015312" rpy="0 0 0"/>
+      <mass value="0.44225"/>
+      <inertia ixx="0.00031483" ixy="-3.882E-08" ixz="3.7547E-08" iyy="0.00016784" iyz="6.6712E-06" izz="0.00035617"/>
     </inertial>
     <visual>
       <origin xyz="0 0 0" rpy="0 0 0"/>
       <geometry>
-        <mesh filename="package://robot_model/meshes/gripper/gripper_body.STL"/>
-      </geometry>
-      <material name="">
-        <color rgba="0.79216 0.81961 0.93333 1"/>
-      </material>
+      <mesh filename="package://robot_model/meshes/gripper/gripper_body.STL"/>
+    </geometry>
+    <material name="">
+      <color rgba="0.79216 0.81961 0.93333 1"/>
+    </material>
     </visual>
-    <collision>
+      <collision>
       <origin xyz="0 0 0" rpy="0 0 0"/>
       <geometry>
-        <mesh filename="package://robot_model/meshes/gripper/gripper_body.STL"/>
-      </geometry>
+      <mesh filename="package://robot_model/meshes/gripper/gripper_body.STL"/>
+    </geometry>
     </collision>
-  </link>
+</link>
 </robot>

File: robot_model/urdf/lego_bot.xacro (robot description, xacro)
@@ -27,5 +27,5 @@
     <parent link="ee_link" />
     <child link = "gripper_body" />
-    <origin xyz="0.06 0.0 0.0" rpy="0.0 -1.57079632679 1.57079632679" />
+    <origin xyz="0.032 0.0 0.0" rpy="0.0 -1.57079632679 1.57079632679" />
   </joint>
   <link name="TCP"/>
