Commit message: off robot 12/5

File: robot_model/urdf/lego_bot.xacro (robot description, xacro)
@@ -46,5 +46,5 @@
     <parent link="table" />
     <child link = "world" />
-    <origin xyz="0.0 0.0 0.0" rpy="0.0 0.0 0.0" />
+    <origin xyz="0.0 0.0 0.04735" rpy="0.0 0.0 0.0" />
   </joint>
 </robot>

Commit message: boatload of small changes

File: robot_model/urdf/lego_bot.xacro (robot description, xacro)
@@ -10,5 +10,5 @@
   <!-- arm -->
   <xacro:arg name="kinematics_config" default="$(find ur_description)/config/ur5_default.yaml"/>
-  <xacro:ur5_robot prefix="" joint_limited="true" shoulder_pan_lower_limit="${-pi}" shoulder_pan_upper_limit="${pi}" shoulder_lift_lower_limit="${-pi}" shoulder_lift_upper_limit="${pi}" elbow_joint_lower_limit="${-pi}" elbow_joint_upper_limit="${pi}" wrist_1_lower_limit="${-pi}" wrist_1_upper_limit="${pi}" wrist_2_lower_limit="${-pi}" wrist_2_upper_limit="${pi}" wrist_3_lower_limit="${-pi}" wrist_3_upper_limit="${pi}" transmission_hw_interface="$(arg transmission_hw_interface)" kinematics_file="${load_yaml('$(arg kinematics_config)')}"/>
+  <xacro:ur5_robot prefix="" joint_limited="true" shoulder_pan_lower_limit="${-pi}" shoulder_pan_upper_limit="${pi}" shoulder_lift_lower_limit="${-pi}" shoulder_lift_upper_limit="${pi}" elbow_joint_lower_limit="${-pi}" elbow_joint_upper_limit="${pi}" wrist_1_lower_limit="${-pi}" wrist_1_upper_limit="${pi}" wrist_2_lower_limit="${-2*pi}" wrist_2_upper_limit="${0}" wrist_3_lower_limit="${0}" wrist_3_upper_limit="${2*pi}" transmission_hw_interface="$(arg transmission_hw_interface)" kinematics_file="${load_yaml('$(arg kinematics_config)')}"/>
   <joint name="world_joint" type="fixed">
   <parent link="world"/>
@@ -39,5 +39,5 @@
   <xacro:include filename="$(find realsense2_description)/urdf/_d435.urdf.xacro"/>
   <sensor_d435 parent="gripper_body">
-    <origin xyz="0  -0.1157 0.03799" rpy="0 0 -1.57079632679"/>
+    <origin xyz="0  -0.11325 0.038" rpy="0 0 -1.57079632679"/>
   </sensor_d435>
     <!-- Table -->
@@ -45,6 +45,6 @@
   <joint name="table_mount_robot" type="fixed">
     <parent link="table" />
-    <child link = "world" />
-    <origin xyz="0.0 0.0 0.04735" rpy="0.0 0.0 0.0" />
+      <child link = "world" />
+      <origin xyz="0.0 0.0 0.0495" rpy="0.0 0.0 0.0" />
   </joint>
 </robot>

Commit message: fix dataextractors and rotation error

File: robot_model/urdf/lego_bot.xacro (robot description, xacro)
@@ -39,5 +39,5 @@
   <xacro:include filename="$(find realsense2_description)/urdf/_d435.urdf.xacro"/>
   <sensor_d435 parent="gripper_body">
-    <origin xyz="0  -0.1157 0.03799" rpy="0 0 -1.57079632679"/>
+    <origin xyz="0  -0.11325 0.038" rpy="0 0 -1.57079632679"/>
   </sensor_d435>
     <!-- Table -->
@@ -46,5 +46,5 @@
     <parent link="table" />
     <child link = "world" />
-    <origin xyz="0.0 0.0 0.04735" rpy="0.0 0.0 0.0" />
+    <origin xyz="0.0 0.0 0.05" rpy="0.0 0.0 0.0" />
   </joint>
 </robot>

Commit message: working calibration

File: robot_model/urdf/lego_bot.xacro (robot description, xacro)
@@ -33,5 +33,5 @@
     <parent link="gripper_body" />
     <child link = "TCP" />
-    <origin xyz="0.0 -0.264 0.0" rpy="3.14159265359 1.57079632679 -1.57079632679" />
+    <origin xyz="0.0 -0.26983 0.0" rpy="3.14159265359 1.57079632679 -1.57079632679" />
   </joint>
   <!-- Realsense Cam -->
